File: KaCat1-2 wiring/KaCat1-2 wiring.kicad_sch (KiCad schematic)
At the start: 6 parts

Commit message: Add files via upload
Parts:
- added U5: ~, symbol Objects:LORA_RadioUnit
- renumbered Out1 to OUT1, S1 to U1, S2 to U2, S3 to U3, S4 to U4
Connections:
- net +3.3V: now also U5. (GND)
- net GND1: now also U5. (GND)
- net RX0: now also MCU1.0 (TX1); no longer MCU1.8 (TX2)
- net RX1: now also MCU1.8 (TX2), U5.A4 (RX)
- net TX0: now also MCU1.1 (RX1); no longer MCU1.7 (RX2)
- net TX1: now also MCU1.7 (RX2), U5.A5 (TX)
- net IO_LED: now reaches MCU1.5
Other:
- removed sheet Radio Unit
- sheet Power supply: file untitled.kicad_sch -> PowerSupply.kicad_sch
- sheet Secondary Mission - LED ports: added IO_LED; removed none
- moved on the sheet: MCU1, OUT1, U1, U2, U3, U4
